File: hw/_module_interface.sch (KiCad schematic (older format))
At the start: 53 parts, among them J1 clock, J10 out7, J11 out8, J2 cv1, J3 cv2, J4 out1, J5 out2, J6 out1, J7 out2, J8 out5, J9 out6, Q1 2SC1815, SW1 command, SW2 enter, U1 OLED_Display_SSD1306

Commit message: hardware: artwork done.
Parts:
- C1, C2: footprint (none) -> Attenuverter:C_Axial_L4.8mm_D2.0mm_P2.54mm_Horizontal
- D1, D2, D3, D4, D5, D6, D7, D8, D9: footprint (none) -> LED_THT:LED_D4.0mm
- J1, J10, J11, J2, J3, J4, J5, J8, J9: footprint (none) -> Attenuverter:mono_jack_3.5mm
- J12: renamed from J?; footprint (none) -> Connector_PinSocket_2.54mm:PinSocket_2x10_P2.54mm_Vertical
- J6: value out1 -> out3; footprint (none) -> Attenuverter:mono_jack_3.5mm
- J7: value out2 -> out4; footprint (none) -> Attenuverter:mono_jack_3.5mm
- Q1: footprint Package_TO_SOT_THT:TO-92_Inline -> Package_TO_SOT_THT:TO-92_Inline_Wide
- R1, R10, R11, R12, R13, R14, R15, R16, R17, R18, R19, R2, R20, R21, R22, R23, R24, R25, R26, R3, R4, R5, R6, R7, R8, R9: footprint (none) -> Resistor_THT:R_Axial_DIN0207_L6.3mm_D2.5mm_P2.54mm_Vertical
- SW1: footprint (none) -> Rotary_Encoder:RotaryEncoder_Alps_EC12E_Vertical_H20mm
- SW2: footprint (none) -> Attenuverter:push_button
- U1: footprint (none) -> Attenuverter:aki_OLED_0.96in
Connections:
- net RE2: now also J12.3 (Pin_3); no longer J12.6 (Pin_6)
- net button: now also J12.5 (Pin_5); no longer J12.8 (Pin_8)
- net clock: now also J12.8 (Pin_8); no longer J12.7 (Pin_7)
- net cv_1_in: now also J12.6 (Pin_6); no longer J12.5 (Pin_5)
- net cv_2_in: now also J12.7 (Pin_7); no longer J12.3 (Pin_3)
- net display_scl: now also J12.1 (Pin_1); no longer J12.2 (Pin_2)
- net display_sda: now also J12.2 (Pin_2); no longer J12.1 (Pin_1)
- net out_1: now also J12.14 (Pin_14); no longer J12.13 (Pin_13)
- net out_2: now also J12.16 (Pin_16); no longer J12.15 (Pin_15)
- net out_3: now also J12.15 (Pin_15); no longer J12.17 (Pin_17)
- net out_4: now also J12.13 (Pin_13); no longer J12.19 (Pin_19)
- net out_5: now also J12.18 (Pin_18); no longer J12.20 (Pin_20)
- net out_6: now also J12.20 (Pin_20); no longer J12.18 (Pin_18)
- net out_7: now also J12.19 (Pin_19); no longer J12.16 (Pin_16)
- net out_8: now also J12.17 (Pin_17); no longer J12.14 (Pin_14)
