File: hw/ModuleMid.kicad_pcb (KiCad board)
At the start: 2 copper layers, 48.3 x 99.1 mm, 23 parts, among them J13 interface_to_mid, J14 mid_to_back_1, J15 mid_to_back_2, U2 MCP4922, U3 RaspberryPi_Pico, U4 MCP4922, U5 MCP4922, U6 MCP4922

Commit message: Software: - Added CV control, but for limited functions. - Added BPM mode.
Hardware:
- Version ordered to Elecrow.
Changed lines of the file:
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@@
     (descr "Diode, DO-35_SOD27 series, Axial, Horizontal, pin pitch=7.62mm, , length*diameter=4*2mm^2, , http://www.diodes.com/_files/packages/DO-35.pdf")
     (tags "Diode DO-35_SOD27 series Axial Horizontal pin pitch 7.62mm  length 4mm diameter 2mm")
-    (fp_text reference D10 (at -2.54 0 90) (layer F.SilkS)
+    (fp_text reference D10 (at -3.81 0 90) (layer F.SilkS)
       (effects (font (size 1 1) (thickness 0.15)))
     )
@@
       (effects (font (size 1 1) (thickness 0.15)))
     )
-    (fp_text user K (at 0 -1.8 90) (layer F.SilkS)
+    (fp_text user K (at -1.27 0 90) (layer F.SilkS)
       (effects (font (size 1 1) (thickness 0.15)))
     )
@@
     (fp_line (start 8.67 1.25) (end 8.67 -1.25) (layer F.CrtYd) (width 0.05))
     (fp_line (start 8.67 -1.25) (end -1.05 -1.25) (layer F.CrtYd) (width 0.05))
-    (fp_text user K (at 0 -1.8 90) (layer F.SilkS)
+    (fp_text user K (at -1.27 0 90) (layer F.SilkS)
       (effects (font (size 1 1) (thickness 0.15)))
     )
@@
     (fp_line (start 8.67 1.25) (end 8.67 -1.25) (layer F.CrtYd) (width 0.05))
     (fp_line (start 8.67 -1.25) (end -1.05 -1.25) (layer F.CrtYd) (width 0.05))
-    (fp_text user K (at 0 -1.8 90) (layer F.SilkS)
+    (fp_text user K (at -1.27 0 90) (layer F.SilkS)
       (effects (font (size 1 1) (thickness 0.15)))
     )
