File: hw/_module_mid.sch (KiCad schematic (older format))
At the start: 20 parts, among them U2 MCP4922, U3 RaspberryPi_Pico, U4 MCP4922, U5 MCP4922, U6 MCP4922

Commit message: hardware: artwork done.
Parts:
- removed J?: interface_to_mid, symbol Connector_Generic:Conn_02x10_Odd_Even
- removed J?: mid_to_back_1, symbol Connector_Generic:Conn_02x08_Odd_Even
- removed J?: mid_to_back_2, symbol Connector_Generic:Conn_02x08_Odd_Even
- added J13: interface_to_mid, Connector_PinSocket_2.54mm:PinSocket_2x10_P2.54mm_Vertical, symbol Connector_Generic:Conn_02x10_Odd_Even
- added J14: mid_to_back_1, Connector_PinHeader_2.54mm:PinHeader_2x08_P2.54mm_Vertical, symbol Connector_Generic:Conn_02x08_Odd_Even
- added J15: mid_to_back_2, Connector_PinHeader_2.54mm:PinHeader_2x08_P2.54mm_Vertical, symbol Connector_Generic:Conn_02x08_Odd_Even
- C10, C4, C6, C8: value 100u -> 10u; footprint (none) -> Capacitor_THT:CP_Radial_D6.3mm_P2.50mm
- C3, C5, C7, C9: footprint (none) -> Attenuverter:C_Axial_L4.8mm_D2.0mm_P2.54mm_Horizontal
- U2, U4, U5, U6: footprint (none) -> Package_DIP:DIP-14_W7.62mm
- U3: footprint (none) -> Attenuverter:Raspberry_Pi_pico_topside_up
Connections:
- net +3V3: now also J13.10 (Pin_10), J13.9 (Pin_9), J14.8 (Pin_8), J15.9 (Pin_9)
- net GND: now also J13.11 (Pin_11), J13.12 (Pin_12), J14.9 (Pin_9), J15.8 (Pin_8)
- net RE1: now also J13.4 (Pin_4)
- net RE2: now also J13.3 (Pin_3)
- net button: now also J13.5 (Pin_5)
- net clock: now also J13.8 (Pin_8)
- net cv1: now also J15.6 (Pin_6)
- net cv2: now also J15.14 (Pin_14)
- net cv_1_in: now also J13.6 (Pin_6), J15.10 (Pin_10)
- net cv_2_in: now also J13.7 (Pin_7), J15.12 (Pin_12)
- net da_cs_2: now also U3.19 (GP14); no longer U3.16 (GP12)
- net da_cs_3: now also U3.20 (GP15); no longer U3.17 (GP13)
- net da_cs_4: now also U3.21 (GP16/SPI_RX); no longer U3.19 (GP14)
- net dac_1_a: now also J14.3 (Pin_3)
- net dac_1_b: now also J14.5 (Pin_5)
- net dac_2_a: now also J14.13 (Pin_13)
- net dac_2_b: now also J14.15 (Pin_15)
- net dac_3_a: now also J15.2 (Pin_2)
- net dac_3_b: now also J15.1 (Pin_1)
- net dac_4_a: now also J15.7 (Pin_7)
- net dac_4_b: now also J15.11 (Pin_11)
- net display_scl: now also J13.1 (Pin_1)
- net display_sda: now also J13.2 (Pin_2)
- net out_1: now also J13.14 (Pin_14), J14.1 (Pin_1)
- net out_2: now also J13.16 (Pin_16), J14.7 (Pin_7)
- net out_3: now also J13.15 (Pin_15), J14.11 (Pin_11)
- net out_4: now also J13.13 (Pin_13), J14.16 (Pin_16)
- net out_5: now also J13.18 (Pin_18), J15.4 (Pin_4)
- net out_6: now also J13.20 (Pin_20), J15.3 (Pin_3)
- net out_7: now also J13.19 (Pin_19), J15.5 (Pin_5)
- net out_8: now also J13.17 (Pin_17), J15.13 (Pin_13)
- net polarity_1: now also J14.2 (Pin_2)
- net polarity_2: now also J14.4 (Pin_4)
- net polarity_3: now also J14.12 (Pin_12)
- net polarity_4: now also J14.14 (Pin_14)
- net polarity_5: now also J14.6 (Pin_6)
- net polarity_6: now also U3.17 (GP13), J14.10 (Pin_10); no longer U3.27 (GP21)
- net polarity_7: now also J15.16 (Pin_16)
- net polarity_8: now also U3.27 (GP21), J15.15 (Pin_15); no longer U3.22 (GP17/SPI_CS)
